File: Hardware/oxgyen_harvester/general_layout.kicad_sch (KiCad schematic)
At the start: 15 parts, among them J1 Barrel_Jack_Switch, J2 Conn_01x20, J3 Conn_01x20, J4 Conn_01x20, J5 OLED, J6 Gas_Pressure_Sensor, J7 Gas_Flowrate_Concentration_Se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, SW1 SW_SPDT, U1 Buck_Converter, U2 Buck_Converter

Commit message: Hardware and software changes
Parts:
- removed J5: OLED, TerminalBlock:TerminalBlock_bornier-5_P5.08mm, symbol Connector:Screw_Terminal_01x05
- added J5: OLED, TerminalBlock:TerminalBlock_bornier-4_P5.08mm, symbol Connector:Screw_Terminal_01x04
Connections:
- net +24V: now also SW1.2 (B); no longer SW1.3 (C)
- net +5V: now also J5.1 (Pin_1)
- net GND: now also SW1.3 (C), J5.2 (Pin_2); no longer SW1.1 (A)
- net OLED_SCL: now also J5.3 (Pin_3)
- net OLED_SDA: now also J5.4 (Pin_4)
- net at J1.1: now also SW1.1 (A); no longer SW1.2 (B)
- net OLED_RST renamed PB2

Commit message: Latest changes in firmware hardware and documentation
Parts:
- J2, J3, J4: footprint Connector_PinHeader_2.54mm:PinHeader_1x20_P2.54mm_Vertical -> Connector_PinSocket_2.54mm:PinSocket_1x20_P2.54mm_Vertical
- SW1: footprint Connector_PinHeader_2.54mm:PinHeader_1x03_P2.54mm_Vertical -> Connector_PinSocket_2.54mm:PinSocket_1x03_P2.54mm_Vertical
Changed lines of the file:
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@@
 			)
 		)
-		(property "Footprint" "Connector_PinHeader_2.54mm:PinHeader_1x03_P2.54mm_Vertical"
+		(property "Footprint" "Connector_PinSocket_2.54mm:PinSocket_1x03_P2.54mm_Vertical"
 			(at 67.31 73.66 0)
 			(effects
@@
 			)
 		)
-		(property "Footprint" "Connector_PinHeader_2.54mm:PinHeader_1x20_P2.54mm_Vertical"
+		(property "Footprint" "Connector_PinSocket_2.54mm:PinSocket_1x20_P2.54mm_Vertical"
 			(at 162.56 88.9 0)
 			(effects
@@
 			)
 		)
-		(property "Footprint" "Connector_PinHeader_2.54mm:PinHeader_1x20_P2.54mm_Vertical"
+		(property "Footprint" "Connector_PinSocket_2.54mm:PinSocket_1x20_P2.54mm_Vertical"
 			(at 148.59 149.86 0)
 			(effects
@@
 			)
 		)
-		(property "Footprint" "Connector_PinHeader_2.54mm:PinHeader_1x20_P2.54mm_Vertical"
+		(property "Footprint" "Connector_PinSocket_2.54mm:PinSocket_1x20_P2.54mm_Vertical"
 			(at 146.05 88.9 0)
 			(effects
